Commit message: Update and add new URDF for current 3DX models

File: urdf/3dx_cs_descr.urdf.xacro (robot description, xacro)
@@ -16,12 +16,12 @@
 OF THIS SOFTWARE, EVEN IF ADVISED OF THE POSSIBILITY OF SUCH DAMAGE.
 -->
-<robot name="numurus_3dx_c" xmlns:xacro="http://ros.org/wiki/xacro">
+<robot name="numurus_3dx_cs" xmlns:xacro="http://ros.org/wiki/xacro">
 <!-- Includes -->
     <xacro:include filename="$(find num_sdk_msgs)/urdf/include/materials.urdf.xacro" />
     <!-- Arguments -->
     <xacro:arg name="camera_name"   default="stereo_cam" />
-    <xacro:arg name="camera_model"  default="zedm" />
+    <xacro:arg name="camera_model"  default="zed2" />
     <xacro:arg name="base_frame"    default="base_link" />
-    <xacro:arg name="cam_pos_x"     default="-0.0294" />
+    <xacro:arg name="cam_pos_x"     default="-0.0316" />
     <xacro:arg name="cam_pos_y"     default="0.0" />
     <xacro:arg name="cam_pos_z"     default="0.0" />
@@ -44,4 +44,5 @@
     <link name="$(arg base_frame)" />
 <!-- pan/tilt TODO -->
+<!-- Lord AHRS TODO -->
 <!-- 3DX Center Joint -->
     <joint name="3dx_center_joint" type="fixed">
@@ -52,7 +53,7 @@
     <link name="3dx_center_frame">
       <visual>
-        <origin xyz="-0.15 0.06 0.026" rpy="-1.57075 0 -1.57075"/>
+        <origin xyz="-0.24 0.095 0.051" rpy="-1.57075 0 -1.57075"/>
         <geometry>
-          <mesh filename="package://num_sdk_msgs/urdf/models/3dx_c.stl" name="3dx_mat" scale="0.001 0.001 0.001"/>
+          <mesh filename="package://num_sdk_msgs/urdf/models/3dx_cw.stl" name="3dx_mat" scale="0.001 0.001 0.001"/>
         </geometry>
         <material name="3dx_mat" />

File: urdf/3dx_cw_descr.urdf.xacro (robot description, xacro)
@@ -16,12 +16,12 @@
 OF THIS SOFTWARE, EVEN IF ADVISED OF THE POSSIBILITY OF SUCH DAMAGE.
 -->
-<robot name="numurus_3dx_c" xmlns:xacro="http://ros.org/wiki/xacro">
+<robot name="numurus_3dx_cw" xmlns:xacro="http://ros.org/wiki/xacro">
 <!-- Includes -->
     <xacro:include filename="$(find num_sdk_msgs)/urdf/include/materials.urdf.xacro" />
     <!-- Arguments -->
     <xacro:arg name="camera_name"   default="stereo_cam" />
-    <xacro:arg name="camera_model"  default="zedm" />
+    <xacro:arg name="camera_model"  default="zed2" />
     <xacro:arg name="base_frame"    default="base_link" />
-    <xacro:arg name="cam_pos_x"     default="-0.0294" />
+    <xacro:arg name="cam_pos_x"     default="-0.0316" />
     <xacro:arg name="cam_pos_y"     default="0.0" />
     <xacro:arg name="cam_pos_z"     default="0.0" />
@@ -52,7 +52,7 @@
     <link name="3dx_center_frame">
       <visual>
-        <origin xyz="-0.15 0.06 0.026" rpy="-1.57075 0 -1.57075"/>
+        <origin xyz="-0.24 0.095 0.051" rpy="-1.57075 0 -1.57075"/>
         <geometry>
-          <mesh filename="package://num_sdk_msgs/urdf/models/3dx_c.stl" name="3dx_mat" scale="0.001 0.001 0.001"/>
+          <mesh filename="package://num_sdk_msgs/urdf/models/3dx_cw.stl" name="3dx_mat" scale="0.001 0.001 0.001"/>
         </geometry>
         <material name="3dx_mat" />
