Commit message: URDF changes for better customer access
Moved all of the dependencies for rendering 3DX in rviz to num_sdk_msgs so that customers have easy access. Now, once they've built num_sdk_msgs and sourced its setup.bash, the rendering will just work for them.

File: urdf/3dx_c_descr.urdf.xacro (robot description, xacro)
@@ -18,5 +18,5 @@
 <robot name="numurus_3dx_c" xmlns:xacro="http://ros.org/wiki/xacro">
 <!-- Includes -->
-    <xacro:include filename="$(find num_sdk_base)/urdf/include/materials.urdf.xacro" />
+    <xacro:include filename="$(find num_sdk_msgs)/urdf/include/materials.urdf.xacro" />
     <!-- Arguments -->
     <xacro:arg name="camera_name"   default="stereo_cam" />
@@ -52,7 +52,7 @@
     <link name="3dx_center_frame">
       <visual>
-        <origin xyz="0 0 0" rpy="0 0 0"/>
+        <origin xyz="-0.15 0.06 0.026" rpy="-1.57075 0 -1.57075"/>
         <geometry>
-          <mesh filename="package://num_sdk_base/urdf/models/3dx_c.stl" name="3dx_mat" scale="0.003 0.003 0.003"/>
+          <mesh filename="package://num_sdk_msgs/urdf/models/3dx_c.stl" name="3dx_mat" scale="0.001 0.001 0.001"/>
         </geometry>
         <material name="3dx_mat" />
@@ -65,13 +65,5 @@
         <origin xyz="$(arg cam_pos_x) $(arg cam_pos_y) $(arg cam_pos_z)" rpy="$(arg cam_roll) $(arg cam_pitch) $(arg cam_yaw)" />
     </joint>
-    <link name="$(arg camera_name)_camera_center">
-        <visual>
-            <origin xyz="0 0 0" rpy="0 0 0"/>
-            <geometry>
-                <mesh filename="package://zed_wrapper/urdf/models/${model}.stl" />
-            </geometry>
-            <material name="${model}_mat" />
-        </visual>
-    </link>
+    <link name="$(arg camera_name)_camera_center"/>
 <!-- Left Camera -->
     <joint name="$(arg camera_name)_left_camera_joint" type="fixed">

Commit message: Changes to support new NEPI-centric names
Huge commit that addresses:
a) New names for projects, repos, filesystem paths, etc. for NEPI
b) Removal of some deprecated source files and related changes

File: urdf/3dx_c_descr.urdf.xacro (robot description, xacro)
@@ -18,5 +18,5 @@
 <robot name="numurus_3dx_c" xmlns:xacro="http://ros.org/wiki/xacro">
 <!-- Includes -->
-    <xacro:include filename="$(find num_sdk_msgs)/urdf/include/materials.urdf.xacro" />
+    <xacro:include filename="$(find nepi_ros_interfaces)/urdf/include/materials.urdf.xacro" />
     <!-- Arguments -->
     <xacro:arg name="camera_name"   default="stereo_cam" />
@@ -54,5 +54,5 @@
         <origin xyz="-0.15 0.06 0.026" rpy="-1.57075 0 -1.57075"/>
         <geometry>
-          <mesh filename="package://num_sdk_msgs/urdf/models/3dx_c.stl" name="3dx_mat" scale="0.001 0.001 0.001"/>
+          <mesh filename="package://nepi_ros_interfaces/urdf/models/3dx_c.stl" name="3dx_mat" scale="0.001 0.001 0.001"/>
         </geometry>
         <material name="3dx_mat" />

File: urdf/3dx_cs_descr.urdf.xacro (robot description, xacro)
@@ -18,5 +18,5 @@
 <robot name="numurus_3dx_cs" xmlns:xacro="http://ros.org/wiki/xacro">
 <!-- Includes -->
-    <xacro:include filename="$(find num_sdk_msgs)/urdf/include/materials.urdf.xacro" />
+    <xacro:include filename="$(find nepi_ros_interfaces)/urdf/include/materials.urdf.xacro" />
     <!-- Arguments -->
     <xacro:arg name="camera_name"   default="stereo_cam" />
@@ -55,5 +55,5 @@
         <origin xyz="-0.24 0.095 0.051" rpy="-1.57075 0 -1.57075"/>
         <geometry>
-          <mesh filename="package://num_sdk_msgs/urdf/models/3dx_cw.stl" name="3dx_mat" scale="0.001 0.001 0.001"/>
+          <mesh filename="package://nepi_ros_interfaces/urdf/models/3dx_cw.stl" name="3dx_mat" scale="0.001 0.001 0.001"/>
         </geometry>
         <material name="3dx_mat" />

File: urdf/3dx_cw_descr.urdf.xacro (robot description, xacro)
@@ -18,5 +18,5 @@
 <robot name="numurus_3dx_cw" xmlns:xacro="http://ros.org/wiki/xacro">
 <!-- Includes -->
-    <xacro:include filename="$(find num_sdk_msgs)/urdf/include/materials.urdf.xacro" />
+    <xacro:include filename="$(find nepi_ros_interfaces)/urdf/include/materials.urdf.xacro" />
     <!-- Arguments -->
     <xacro:arg name="camera_name"   default="stereo_cam" />
@@ -54,5 +54,5 @@
         <origin xyz="-0.24 0.095 0.051" rpy="-1.57075 0 -1.57075"/>
         <geometry>
-          <mesh filename="package://num_sdk_msgs/urdf/models/3dx_cw.stl" name="3dx_mat" scale="0.001 0.001 0.001"/>
+          <mesh filename="package://nepi_ros_interfaces/urdf/models/3dx_cw.stl" name="3dx_mat" scale="0.001 0.001 0.001"/>
         </geometry>
         <material name="3dx_mat" />
